File: projects/vacuum-controller-rev-a/vacuum-controller-rev-a.brd (EAGLE design)
At the start: 56.5 x 56.5 mm, 24 parts, among them J1 MJ-3536N, J2 39512-1006, U1 TPS709, U2 ATTINY85-20SU, U3 SZNUD3124, U4 SN74AHC1G14DCK

Commit message: Starting to tweak the board layout to better suit the enclosure, as well as getting the 3D models of the connectors.
Parts:
- moved J2 3.81 mm to (28.2, 4.19)
Routing:
- net +12V: track 30.5 -> 34.8 mm
- net VAC_CONTROL: track 10.3 -> 14.1 mm
- net AIR_CONTROL: track 8.30 -> 12.1 mm
- net PEDAL_INPUT: track 24.4 -> 26.9 mm
Changed lines of the file:
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@@
 <setting verticaltext="up"/>
 </settings>
-<grid distance="5" unitdist="mil" unit="mil" style="lines" multiple="1" display="no" altdistance="0.025" altunitdist="inch" altunit="inch"/>
+<grid distance="10" unitdist="mil" unit="mil" style="lines" multiple="1" display="no" altdistance="0.025" altunitdist="inch" altunit="inch"/>
 <layers>
 <layer number="1" name="Top" color="4" fill="1" visible="yes" active="yes"/>
@@
 <attribute name="PN" value="MJ-3536N" x="10.541" y="28.2194" size="1.778" layer="27" display="off"/>
 </element>
-<element name="J2" library="molex" package="39512-1006" value="39512-1006" x="28.2194" y="8.001" smashed="yes">
-<attribute name="NAME" x="14.6304" y="11.176" size="1.27" layer="25" font="vector"/>
-<attribute name="MATES" value="39510-0006" x="28.2194" y="8.001" size="1.778" layer="27" display="off"/>
-<attribute name="PN" value="39512-1006" x="28.2194" y="8.001" size="1.778" layer="27" display="off"/>
+<element name="J2" library="molex" package="39512-1006" value="39512-1006" x="28.2194" y="4.191" smashed="yes">
+<attribute name="NAME" x="14.6304" y="7.366" size="1.27" layer="25" font="vector"/>
+<attribute name="MATES" value="39510-0006" x="28.2194" y="4.191" size="1.778" layer="27" display="off"/>
+<attribute name="PN" value="39512-1006" x="28.2194" y="4.191" size="1.778" layer="27" display="off"/>
 </element>
 <element name="R1" library="passives" package="R0402" value="100K" x="27.432" y="29.845" smashed="yes">
@@
 <vertex x="29.337" y="19.177"/>
 <vertex x="23.241" y="19.177"/>
-<vertex x="23.241" y="12.065"/>
-<vertex x="29.337" y="12.065"/>
+<vertex x="23.241" y="8.255"/>
+<vertex x="29.337" y="8.255"/>
 </polygon>
 <via x="23.749" y="14.605" extent="1-16" drill="0.3302"/>
@@
 <contactref element="J2" pad="P$4"/>
 <wire x1="27.239" y1="13.913" x2="29.267" y2="13.913" width="0.4064" layer="1"/>
-<wire x1="30.1244" y1="8.001" x2="30.1244" y2="13.0556" width="0.4064" layer="1"/>
+<wire x1="30.1244" y1="4.191" x2="30.1244" y2="13.0556" width="0.4064" layer="1"/>
 <wire x1="30.1244" y1="13.0556" x2="29.267" y2="13.913" width="0.4064" layer="1"/>
 </signal>
@@
 <wire x1="25.339" y1="16.195" x2="24.765" y2="15.621" width="0.4064" layer="1"/>
 <wire x1="24.765" y1="15.621" x2="23.368" y2="15.621" width="0.4064" layer="1"/>
-<wire x1="22.5044" y1="8.001" x2="22.5044" y2="14.7574" width="0.4064" layer="1"/>
+<wire x1="22.5044" y1="4.191" x2="22.5044" y2="14.7574" width="0.4064" layer="1"/>
 <wire x1="22.5044" y1="14.7574" x2="23.368" y2="15.621" width="0.4064" layer="1"/>
 </signal>
@@
 <contactref element="J2" pad="P$5"/>
 <contactref element="F1" pad="1"/>
-<wire x1="28.6004" y1="5.715" x2="26.3144" y2="8.001" width="1.524" layer="1"/>
-<wire x1="26.3144" y1="8.001" x2="26.289" y2="8.001" width="1.524" layer="1"/>
-<wire x1="26.289" y1="8.001" x2="23.876" y2="5.588" width="1.524" layer="1"/>
-<wire x1="23.876" y1="5.588" x2="21.1074" y2="5.588" width="1.524" layer="1"/>
-<wire x1="21.1074" y1="5.588" x2="18.6944" y2="8.001" width="1.524" layer="1"/>
-<wire x1="28.6004" y1="5.715" x2="31.6484" y2="5.715" width="1.524" layer="1"/>
-<wire x1="31.6484" y1="5.715" x2="33.9344" y2="8.001" width="1.524" layer="1"/>
-<wire x1="33.9344" y1="8.001" x2="33.9344" y2="13.4874" width="1.016" layer="1"/>
+<wire x1="33.9344" y1="4.191" x2="33.9344" y2="13.4874" width="1.016" layer="1"/>
 <wire x1="33.9344" y1="13.4874" x2="35.052" y2="14.605" width="1.016" layer="1"/>
 <wire x1="35.052" y1="14.605" x2="39.359" y2="14.605" width="1.016" layer="1"/>
+<wire x1="33.9344" y1="4.191" x2="33.909" y2="4.191" width="1.27" layer="16"/>
+<wire x1="33.909" y1="4.191" x2="31.242" y2="6.858" width="1.27" layer="16"/>
+<wire x1="31.242" y1="6.858" x2="28.9814" y2="6.858" width="1.27" layer="16"/>
+<wire x1="28.9814" y1="6.858" x2="26.3144" y2="4.191" width="1.27" layer="16"/>
+<wire x1="26.3144" y1="4.191" x2="26.289" y2="4.191" width="1.27" layer="16"/>
+<wire x1="26.289" y1="4.191" x2="23.622" y2="6.858" width="1.27" layer="16"/>
+<wire x1="23.622" y1="6.858" x2="21.3614" y2="6.858" width="1.27" layer="16"/>
+<wire x1="21.3614" y1="6.858" x2="18.6944" y2="4.191" width="1.27" layer="16"/>
 </signal>
 <signal name="PEDAL_DEBOUNCED">
@@
 <wire x1="25.654" y1="29.817" x2="26.924" y2="29.817" width="0.1524" layer="1"/>
 <wire x1="26.924" y1="29.817" x2="26.952" y2="29.845" width="0.1524" layer="1"/>
-<wire x1="4.941" y1="28.2194" x2="4.9784" y2="28.2194" width="0.1524" layer="1"/>
+<wire x1="2.441" y1="28.2194" x2="4.9784" y2="28.2194" width="0.1524" layer="1"/>
 <wire x1="4.9784" y1="28.2194" x2="8.128" y2="31.369" width="0.1524" layer="1"/>
 <wire x1="8.128" y1="31.369" x2="24.892" y2="31.369" width="0.1524" layer="1"/>

Commit message: Many changes to the schematic/board.
- added part numbers to all components
- added 2x470uF electrolytic caps to smooth the 12V rail during relay
  switching events
- switched to a DIP-8 footprint for the ATtiny so we can program it in a
  cheapo programmer and not have to mess around with SOIC clips and all
  that
Parts:
- added C7, C8: 470uF, passives:RADIAL-D8-P3.5-PD0.5
- U1: value TPS709 -> TPS70950
- U2: value ATTINY85-20SU -> ATTINY85-20PU; device atmel:EIAJ-SOIC-8 -> atmel:PDIP-8
- moved C4 9.12 mm to (46.4, 28.7), turned to 0 degrees
- moved C2 6.99 mm to (46.7, 27.1), turned to 0 degrees
- moved U$5 5.45 mm to (23.4, 46.6)
- moved U$7 5.39 mm to (50.6, 33.6)
- moved C3 4.19 mm to (46.7, 24.9), turned to 0 degrees
- moved U2 3.37 mm to (37.0, 28.7), turned to 180 degrees
- moved D2 2.79 mm to (39.0, 20.4)
- moved F1 2.79 mm to (40.3, 17.4)
- moved C1 2.67 mm to (43.9, 21.0), turned to 90 degrees
- moved U1 2.50 mm to (46.7, 21.5), turned to 0 degrees
- moved U4 0.51 mm to (27.8, 27.7)
- moved C5 0.51 mm to (25.1, 27.2)
- moved C6 0.51 mm to (28.7, 30.4)
- moved R1 0.51 mm to (26.9, 29.8)
- moved R2 0.51 mm to (25.1, 29.3)
Connections:
- net PEDAL_INPUT renamed PEDAL_IN
- net +12V: now also C7.+, C8.+
- net +5V: now also U2.P$8; no longer U2.8
- net AGND: now also C7.-, C8.-, U2.P$4; no longer U2.4
- net N$4: now also U2.P$6; no longer U2.6
- net N$6: now also U2.P$5; no longer U2.5
- net PEDAL_DEBOUNCED: now also U2.P$7; no longer U2.7
Routing:
- net +12V: track 34.8 -> 46.3 mm
- net PEDAL_DEBOUNCED: track 7.31 -> 11.2 mm
- net +5V: track 28.1 -> 31.6 mm
- net PEDAL_IN: track 26.9 -> 23.5 mm
- net N$4: track 16.1 -> 18.7 mm
- net N$1: track 6.52 -> 4.35 mm
- net AGND: track 13.2 -> 11.5 mm, vias 25 -> 24

Commit message: Some small tweaks to the grounding for the load driver.
Routing:
- net N$6: track 12.8 -> 14.6 mm
- net AGND: vias 24 -> 38
Other:
- board text added: "Manual Pick and Place Vacuum Controller, rev A Nuclear Furnace, 2017 (tm)"
- board text removed: "Manual Pick and Place Vacuum Controller V1 Nuclear Furnace, 2017 (tm)"
Changed lines of the file:
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@@
 <wire x1="4.5466" y1="7.9502" x2="7.9502" y2="4.5466" width="0" layer="20" curve="-90"/>
 <text x="14.478" y="36.83" size="1.524" layer="25" font="vector" ratio="15">Manual Pick and Place
-Vacuum Controller V1
+Vacuum Controller, rev A
 Nuclear Furnace, 2017 (tm)</text>
 </plain>
@@
 </element>
 <element name="U3" library="on-semiconductor" package="SOT-457" value="SZNUD3124" x="26.289" y="15.113" smashed="yes" rot="R90">
-<attribute name="NAME" x="25.908" y="18.796" size="1.27" layer="25" font="vector" rot="R180"/>
+<attribute name="NAME" x="24.511" y="17.145" size="1.27" layer="25" font="vector" rot="R180"/>
 <attribute name="PN" value="SZNUD3124DMT1G" x="26.289" y="15.113" size="1.778" layer="27" rot="R90" display="off"/>
 </element>
@@
 <vertex x="0" y="1.27"/>
 </polygon>
-<polygon width="0.1524" layer="1" thermals="no">
-<vertex x="29.337" y="19.177"/>
-<vertex x="23.241" y="19.177"/>
-<vertex x="23.241" y="8.255"/>
-<vertex x="29.337" y="8.255"/>
+<polygon width="0.1524" layer="1" isolate="0.254" thermals="no">
+<vertex x="30.353" y="20.066"/>
+<vertex x="23.241" y="20.066"/>
+<vertex x="23.241" y="10.795"/>
+<vertex x="30.353" y="10.795"/>
 </polygon>
 <via x="23.749" y="14.605" extent="1-16" drill="0.3302"/>
@@
 <via x="26.797" y="12.573" extent="1-16" drill="0.3302"/>
 <via x="28.829" y="12.573" extent="1-16" drill="0.3302"/>
-<via x="28.829" y="17.653" extent="1-16" drill="0.3302"/>
-<via x="28.829" y="16.637" extent="1-16" drill="0.3302"/>
-<via x="27.813" y="17.653" extent="1-16" drill="0.3302"/>
-<via x="26.797" y="17.653" extent="1-16" drill="0.3302"/>
-<via x="28.829" y="18.669" extent="1-16" drill="0.3302"/>
-<via x="27.813" y="18.669" extent="1-16" drill="0.3302"/>
-<via x="26.797" y="18.669" extent="1-16" drill="0.3302"/>
+<via x="28.575" y="17.653" extent="1-16" drill="0.3302"/>
+<via x="28.575" y="16.637" extent="1-16" drill="0.3302"/>
+<via x="27.559" y="17.653" extent="1-16" drill="0.3302"/>
+<via x="27.559" y="19.685" extent="1-16" drill="0.3302"/>
+<via x="28.575" y="18.669" extent="1-16" drill="0.3302"/>
+<via x="27.559" y="18.669" extent="1-16" drill="0.3302"/>
+<via x="26.543" y="18.669" extent="1-16" drill="0.3302"/>
 <via x="27.813" y="12.573" extent="1-16" drill="0.3302"/>
 <wire x1="46.736" y1="20.113" x2="46.736" y2="21.463" width="0.508" layer="1"/>
@@
 <contactref element="C8" pad="-"/>
 <contactref element="C7" pad="-"/>
+<via x="29.591" y="16.637" extent="1-16" drill="0.3302"/>
+<via x="29.591" y="17.653" extent="1-16" drill="0.3302"/>
+<via x="29.591" y="18.669" extent="1-16" drill="0.3302"/>
+<via x="23.749" y="11.557" extent="1-16" drill="0.3302"/>
+<via x="24.765" y="11.557" extent="1-16" drill="0.3302"/>
+<via x="25.781" y="11.557" extent="1-16" drill="0.3302"/>
+<via x="26.797" y="11.557" extent="1-16" drill="0.3302"/>
+<via x="27.813" y="11.557" extent="1-16" drill="0.3302"/>
+<via x="28.829" y="11.557" extent="1-16" drill="0.3302"/>
+<via x="29.591" y="19.685" extent="1-16" drill="0.3302"/>
+<via x="28.575" y="19.685" extent="1-16" drill="0.3302"/>
+<via x="28.575" y="15.621" extent="1-16" drill="0.3302"/>
+<via x="29.591" y="15.621" extent="1-16" drill="0.3302"/>
+<via x="26.543" y="19.685" extent="1-16" drill="0.3302"/>
 </signal>
 <signal name="N$6">
 <contactref element="U3" pad="5"/>
 <contactref element="U2" pad="P$5"/>
-<wire x1="26.289" y1="16.313" x2="26.289" y2="16.891" width="0.2032" layer="1"/>
-<wire x1="26.289" y1="16.891" x2="25.781" y2="17.399" width="0.2032" layer="1"/>
-<wire x1="25.781" y1="17.399" x2="25.781" y2="19.177" width="0.2032" layer="1"/>
-<wire x1="25.781" y1="19.177" x2="31.496" y2="24.892" width="0.2032" layer="1"/>
-<wire x1="31.496" y1="24.892" x2="33.147" y2="24.892" width="0.2032" layer="1"/>
+<wire x1="26.289" y1="16.313" x2="26.289" y2="16.764" width="0.1524" layer="1"/>
+<wire x1="26.289" y1="16.764" x2="26.035" y2="17.018" width="0.1524" layer="1"/>
+<wire x1="26.035" y1="17.018" x2="25.527" y2="17.018" width="0.1524" layer="1"/>
+<wire x1="25.527" y1="17.018" x2="25.273" y2="17.272" width="0.1524" layer="1"/>
+<wire x1="25.273" y1="17.272" x2="25.273" y2="20.447" width="0.1524" layer="1"/>
+<wire x1="33.147" y1="24.892" x2="29.718" y2="24.892" width="0.1524" layer="1"/>
+<wire x1="29.718" y1="24.892" x2="25.273" y2="20.447" width="0.1524" layer="1"/>
 </signal>
 <signal name="AIR_CONTROL">
@@
 <contactref element="U3" pad="2"/>
 <contactref element="U2" pad="P$6"/>
-<wire x1="26.289" y1="13.913" x2="26.289" y2="14.605" width="0.2032" layer="1"/>
-<wire x1="26.289" y1="14.605" x2="26.67" y2="14.986" width="0.2032" layer="1"/>
-<wire x1="26.67" y1="14.986" x2="30.988" y2="14.986" width="0.2032" layer="1"/>
-<wire x1="35.687" y1="24.892" x2="35.687" y2="22.987" width="0.2032" layer="1"/>
-<wire x1="35.687" y1="22.987" x2="35.052" y2="22.352" width="0.2032" layer="1"/>
-<wire x1="35.052" y1="22.352" x2="32.893" y2="22.352" width="0.2032" layer="1"/>
-<wire x1="32.893" y1="22.352" x2="32.004" y2="21.463" width="0.2032" layer="1"/>
-<wire x1="32.004" y1="21.463" x2="32.004" y2="16.002" width="0.2032" layer="1"/>
-<wire x1="32.004" y1="16.002" x2="30.988" y2="14.986" width="0.2032" layer="1"/>
+<wire x1="35.687" y1="24.892" x2="35.687" y2="22.987" width="0.1524" layer="1"/>
+<wire x1="35.687" y1="22.987" x2="35.052" y2="22.352" width="0.1524" layer="1"/>
+<wire x1="35.052" y1="22.352" x2="32.893" y2="22.352" width="0.1524" layer="1"/>
+<wire x1="32.893" y1="22.352" x2="32.004" y2="21.463" width="0.1524" layer="1"/>
+<wire x1="32.004" y1="21.463" x2="32.004" y2="15.113" width="0.1524" layer="1"/>
+<wire x1="26.289" y1="13.913" x2="26.289" y2="13.97" width="0.1524" layer="1"/>
+<wire x1="26.289" y1="13.97" x2="26.924" y2="14.605" width="0.1524" layer="1"/>
+<wire x1="26.924" y1="14.605" x2="31.496" y2="14.605" width="0.1524" layer="1"/>
+<wire x1="31.496" y1="14.605" x2="32.004" y2="15.113" width="0.1524" layer="1"/>
 </signal>
 </signals>
