File: projects/vacuum-controller-rev-a/vacuum-controller-rev-a.sch (EAGLE design)
At the start: 24 parts, among them J1 MJ-3536N, J2 39512-1006, U1 TPS709, U2 ATTINY85-20SU, U3 SZNUD3124, U4 SN74AHC1G14DCK

Commit message: Many changes to the schematic/board.
- added part numbers to all components
- added 2x470uF electrolytic caps to smooth the 12V rail during relay
  switching events
- switched to a DIP-8 footprint for the ATtiny so we can program it in a
  cheapo programmer and not have to mess around with SOIC clips and all
  that
Parts:
- added C7, C8: 470uF, passives:CAPACITOR-POLARIZED-RADIAL-D8-P3.5-PD0.5
- C1, C2: PN (none) -> GRM188R61E105KA12D
- C3: PN (none) -> GRM21BR61A106KE19L
- C4, C5, C6: PN (none) -> GRM155R71H104KE14D
- R1: PN (none) -> RC0402FR-07100KL
- R2: PN (none) -> RC0402FR-0710KL
- U1: value TPS709 -> TPS70950
- U2: value ATTINY85-20SU -> ATTINY85-20PU; device atmel:ATTINY85-20SU -> atmel:ATTINY85-20PU
Connections:
- net PEDAL_INPUT renamed PEDAL_IN
- net +12V: now also C7.+, C8.+
- net AGND: now also C7.-, C8.-
Other:
- moved on the sheet: C5, J1, J2, R1, R2, U4A
